File: kicad/tessract.kicad_pcb (KiCad board)
At the start: 2 copper layers, 35 x 50 mm, 23 parts, among them Q1 DMP1045U, U1 MICRO-B_USB, U2 MCP73832T, U3 MCP1755, U4 ATMEL_ATTINY85_20SU, U5 OSRAM_LRTB_GFTG, U6 HM-10

Commit message: copper plane
Routing:
- added copper zone on F.Cu, net Earth
